File: geiger.kicad_pcb (KiCad board)
At the start: 2 copper layers, 117 x 74 mm, 37 parts, among them J1 Screw_Terminal_01x02, SW1 SW_SPST, T1 IRFP450, T2 P55NF06, T3 BC517, U1 NE555P, U2 LM336Z25, U3 LM311, U4 STEP-DOWN-5V, U5 nodemcu-esp32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

Commit message: Traces and footprint fix
Parts:
- added R40: 100k, Resistor_THT:R_Axial_DIN0207_L6.3mm_D2.5mm_P7.62mm_Horizontal, F.Cu at (53.6, 170.8)
Routing:
- net Net-(R40-Pad1): track 11.9 -> 15.7 mm

Commit message: Miller capacitance discharge fix
Parts:
- R40: value 100k -> 1.5k

Commit message: T symbol fixes
Parts:
- U5: footprint geiger:nodemcu32_zwyczajowy -> geiger:NODEMCU_ESP32
Connections:
- T1 pad 1: Net-(D1-Pad2) -> Net-(R40-Pad1)
- T1 pad 2: Net-(R40-Pad1) -> Net-(D1-Pad2)
- T2 pad 1: Net-(T2-Pad1) -> Net-(R4-Pad1)
- T2 pad 2: Net-(R4-Pad1) -> Net-(T2-Pad2)
- U1 pad 3: Net-(T2-Pad1) -> Net-(T2-Pad2)
Routing:
- net GND: track 35.1 -> 20.9 mm
- net Net-(T2-Pad1): track 13.2 -> 0.00 mm
- net Net-(T2-Pad2): track 0.00 -> 12.1 mm
- net Net-(R40-Pad1): track 15.7 -> 11.8 mm
- net +8V: track 176.1 -> 178.2 mm
- net Net-(D1-Pad2): track 31.6 -> 33.3 mm
- net Net-(R4-Pad1): track 27.3 -> 26.3 mm
- net Net-(C2-Pad2): track 27.8 -> 27.0 mm

Commit message: T1 modernized
Parts:
- T1: value IRFP450 -> IPAN70R450P7S
