File: geiger.sch (KiCad schematic (older format))
At the start: 37 parts, among them SW1 SW_SPST, T1 IRFP450, T2 P55NF06, T3 BC517, U1 NE555P, U2 LM336Z25, U3 LM311, U4 STEP-DOWN-5V, U5 nodemcu-esp32, U6 GEIGERTUBE-STS6

Commit message: a
Parts:
- U2: symbol Reference_Voltage:LM385Z-2.5 -> geiger-rescue:LM385Z-2.5-Reference_Voltage
Connections:
- net GND: now also U2.1 (A); no longer U2.3 (A)
Changed lines of the file:
@@
 $EndComp
 $Comp
-L Reference_Voltage:LM385Z-2.5 U2
+L geiger-rescue:LM385Z-2.5-Reference_Voltage U2
 U 1 1 60821F46
 P 3650 5600

Commit message: Better connectors and minor trace improvements.
Parts:
- removed BT1: 2X18650 series, Connector_PinHeader_2.54mm:PinHeader_1x02_P2.54mm_Vertical, symbol Device:Battery
- added J1: Screw_Terminal_01x02, TerminalBlock:TerminalBlock_Altech_AK300-2_P5.00mm, symbol Connector:Screw_Terminal_01x02
- U6: footprint Connector_PinSocket_2.54mm:PinSocket_1x02_P2.54mm_Vertical -> TerminalBlock:TerminalBlock_Altech_AK300-2_P5.00mm
Connections:
- net GND: now also J1.1 (Pin_1)
- net at SW1.1 (A): now also J1.2 (Pin_2)
Changed lines of the file:
@@
 F 0 "U6" H 3700 4065 50  0000 C CNN
 F 1 "GEIGERTUBE-STS6" H 3700 3974 50  0000 C CNN
-F 2 "Connector_PinSocket_2.54mm:PinSocket_1x02_P2.54mm_Vertical" H 3700 3800 50  0001 C CNN
+F 2 "TerminalBlock:TerminalBlock_Altech_AK300-2_P5.00mm" H 3700 3800 50  0001 C CNN
 F 3 "" H 3700 3800 50  0001 C CNN
 	1    3700 3800
@@
 $EndComp
 $Comp
-L Device:Battery BT1
-U 1 1 607C6CDB
-P 950 1500
-F 0 "BT1" H 1050 1600 50  0000 L CNN
-F 1 "2X18650 series" H 950 1500 50  0000 L CNN
-F 2 "Connector_PinHeader_2.54mm:PinHeader_1x02_P2.54mm_Vertical" V 950 1560 50  0001 C CNN
-F 3 "~" V 950 1560 50  0001 C CNN
-	1    950  1500
-	1    0    0    -1
-$EndComp
+L Connector:Screw_Terminal_01x02 J1
+U 1 1 6080789A
+P 750 1550
+F 0 "J1" H 668 1225 50  0000 C CNN
+F 1 "Screw_Terminal_01x02" H 668 1316 50  0000 C CNN
+F 2 "TerminalBlock:TerminalBlock_Altech_AK300-2_P5.00mm" H 750 1550 50  0001 C CNN
+F 3 "~" H 750 1550 50  0001 C CNN
+	1    750  1550
+	-1   0    0    1
+$EndComp
+Wire Wire Line
+	950  1550 950  1700
+Wire Wire Line
+	950  1450 950  1300
 $EndSCHEMATC

Commit message: T1 gate fix
Parts:
- added R40: 100k, symbol Device:R_Small
Connections:
- net GND: now also R40.2
- net at T1.1 (G), T2.3 (S): now also R40.1

Commit message: Traces and footprint fix
Parts:
- R40: footprint (none) -> Resistor_THT:R_Axial_DIN0207_L6.3mm_D2.5mm_P7.62mm_Horizontal
Changed lines of the file:
@@
 F 0 "R40" V 854 4250 50  0000 C CNN
 F 1 "100k" V 945 4250 50  0000 C CNN
-F 2 "" H 1050 4250 50  0001 C CNN
+F 2 "Resistor_THT:R_Axial_DIN0207_L6.3mm_D2.5mm_P7.62mm_Horizontal" H 1050 4250 50  0001 C CNN
 F 3 "~" H 1050 4250 50  0001 C CNN
 	1    1050 4250
@@
 Connection ~ 1150 4250
 $Comp
-L power:GND #PWR?
+L power:GND #PWR0118
 U 1 1 60864467
 P 950 4250
-F 0 "#PWR?" H 950 4000 50  0001 C CNN
+F 0 "#PWR0118" H 950 4000 50  0001 C CNN
 F 1 "GND" H 955 4077 50  0000 C CNN
 F 2 "" H 950 4250 50  0001 C CNN

Commit message: Miller capacitance discharge fix
Parts:
- R40: value 100k -> 1.5k
Changed lines of the file:
@@
 P 1050 4250
 F 0 "R40" V 854 4250 50  0000 C CNN
-F 1 "100k" V 945 4250 50  0000 C CNN
+F 1 "1.5k" V 945 4250 50  0000 C CNN
 F 2 "Resistor_THT:R_Axial_DIN0207_L6.3mm_D2.5mm_P7.62mm_Horizontal" H 1050 4250 50  0001 C CNN
 F 3 "~" H 1050 4250 50  0001 C CNN

Commit message: T symbol fixes
Parts:
- U5: footprint geiger:nodemcu32_zwyczajowy -> geiger:NODEMCU_ESP32
Changed lines of the file:
@@
 F 0 "U5" H 8025 6525 50  0000 C CNN
 F 1 "nodemcu-esp32" H 8025 6434 50  0000 C CNN
-F 2 "geiger:nodemcu32_zwyczajowy" H 6900 7000 50  0001 C CNN
+F 2 "geiger:NODEMCU_ESP32" H 6900 7000 50  0001 C CNN
 F 3 "" H 6900 7000 50  0001 C CNN
 	1    8100 5350

Commit message: T1 modernized
Parts:
- T1: value IRFP450 -> IPAN70R450P7S
Changed lines of the file:
@@
 P 1350 4250
 F 0 "T1" H 1554 4296 50  0000 L CNN
-F 1 "IRFP450" H 1554 4205 50  0000 L CNN
+F 1 "IPAN70R450P7S" H 1554 4205 50  0000 L CNN
 F 2 "Package_TO_SOT_THT:TO-247-3_Vertical" H 1550 4350 50  0001 C CNN
 F 3 "~" H 1350 4250 50  0001 C CNN
